File: hardware/WO30109_FreshAir/WO30109_FreshAir.kicad_pcb (KiCad board)
At the start: 2 copper layers, 63.4 x 83.1 mm, 59 parts, among them K1 G5Q-1 DC12, K2 G5Q-1 DC12, K3 G5Q-1 DC12, K4 G5Q-1 DC12, P1 AC IN 230V, P2 PROG, P3 AC OUT, Q1 Si2302CDS, Q2 Si2302CDS, Q3 Si2302CDS, Q4 Si2302CDS, U1 ESP32-C6-WROOM-1-N8, U2 IRM-02-12, U3 SYN480R, U4 AP63203WU-7, Y1 13.52127MHz 20pF

Commit message: hw: V3.2 4 路光耦 DI 輸入、拿掉指撥，上緣加長 10mm
- J5 7P 3.5mm 插拔端子：+12V（R23 1.5k 限流，短路 8mA）／IN1–IN4／COM／GND
- U5 TLP290-4 交流輸入光耦 ×4（乾接點、5–24VDC、NPN/PNP 都可），R15–R18 3.3k，C18–C21 10nF
- DI1–4 → IO22/IO21/IO20/IO19（內建上拉）；S1 指撥拿掉
- scripts/upgrade_v32_pcb.py：從 V3.1 PCB 重建，A* 佈新網路（不動既有走線、繞開 433 匹配區、
  長線自動試佈線順序、新區域縫合與孤島接回）
- mains_router：stamp_r、keep_cl、封裝內建禁佈區、set_board（預設值維持舊行為）
- add_stitching：STITCH_REGION、--islands；assign_3d 冪等；7P 端子封裝與 3D 模型
- ERC 0；DRC 錯誤 0、未連線 0、parity 0；CPL 測試 OK

Co-Authored-By: Claude Opus 5.5 (1M context) <noreply@anthropic.com>
Parts:
- removed S1: DIP 2P, Button_Switch_SMD:SW_DIP_SPSTx02_Slide_Copal_CHS-02B_W7.62mm_P1.27mm
- added C18: 10nF, Capacitor_SMD:C_0603_1608Metric, B.Cu at (110.1, 111.6)
- added C19: 10nF, Capacitor_SMD:C_0603_1608Metric, B.Cu at (112.6, 111.6)
- added C20: 10nF, Capacitor_SMD:C_0603_1608Metric, B.Cu at (115.1, 111.6)
- added C21: 10nF, Capacitor_SMD:C_0603_1608Metric, B.Cu at (117.7, 111.6)
- added J5: DI 12V/IN1-4/COM/GND, WOOW:TerminalBlock_Pluggable_1x07_P3.50mm_Horizontal, F.Cu at (113.0, 97.5)
- added R15: 3.3k, Resistor_SMD:R_1206_3216Metric, B.Cu at (106.0, 93.5)
- added R16: 3.3k, Resistor_SMD:R_1206_3216Metric, B.Cu at (109.5, 93.5)
- added R17: 3.3k, Resistor_SMD:R_1206_3216Metric, B.Cu at (113.0, 93.5)
- added R18: 3.3k, Resistor_SMD:R_1206_3216Metric, B.Cu at (116.5, 93.5)
- added R23: 1.5k, Resistor_SMD:R_1206_3216Metric, B.Cu at (102.5, 93.5)
- added U5: TLP290-4, Package_SO:SOP-16_4.55x10.3mm_P1.27mm, B.Cu at (114.5, 104.9)
Connections:
- U1 pad 11: /Mode_bit0 -> unconnected-(U1-IO10-Pad11)
- U1 pad 12: /Mode_bit1 -> unconnected-(U1-IO11-Pad12)
- U1 pad 17: unconnected-(U1-IO19-Pad17) -> /DI_4
- U1 pad 18: unconnected-(U1-IO20-Pad18) -> /DI_3
- U1 pad 19: unconnected-(U1-IO21-Pad19) -> /DI_2
- U1 pad 20: unconnected-(U1-IO22-Pad20) -> /DI_1
Routing:
- net /+12V: track 66.1 -> 137.3 mm, vias 1 -> 5
- net /Mode_bit0: track 45.6 -> 0.00 mm, vias 1 -> 0
- net /Mode_bit1: track 44.8 -> 0.00 mm, vias 1 -> 0
- net /DI_4: track 0.00 -> 27.6 mm, vias 0 -> 3
- net /DI_2: track 0.00 -> 26.2 mm, vias 0 -> 3
- net /DI_1: track 0.00 -> 23.3 mm, vias 0 -> 1
- net /DI_3: track 0.00 -> 22.5 mm, vias 0 -> 1
- net /GND: track 265.8 -> 245.5 mm, vias 100 -> 126
- net /DI_COM: track 0.00 -> 19.7 mm, vias 0 -> 3
- net /DI_A1: track 0.00 -> 11.3 mm
- net /DI_A2: track 0.00 -> 10.9 mm
- net /DI_A3: track 0.00 -> 10.5 mm
- net /DI_A4: track 0.00 -> 10.3 mm
- net /DI_IN4: track 0.00 -> 2.50 mm
- net /DI_IN3: track 0.00 -> 2.50 mm
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Other:
- board size 63.4 x 83.1 mm -> 63.4 x 93.1 mm
- board text added: "12V"
- board text added: "COM"
- board text added: "GND"
- board text added: "IN1"
- board text added: "IN2"
- board text added: "IN3"
- board text added: "IN4"

Commit message: fix(V3.2): 板框改 L 形，P1（AC IN）前方維持原板緣
第一版 V3.2 上緣整片加長 10mm，P1 開口朝板邊的插拔座前方多了一塊板子，
插頭與 230V 電線會壓在低壓 GND 鋪銅上方（空氣間隙遠小於 6.4mm 加強絕緣）。
DRC 只量銅箔間距，看不到插頭。改成只加長 J5 那一段（x 100–125.9），
確認 P1 前方無走線、過孔、鋪銅；DRC 錯誤 0、未連線 0、parity 0。

Co-Authored-By: Claude Opus 5.5 (1M context) <noreply@anthropic.com>
Routing:
- net /GND: vias 126 -> 124
Other:
- outline, holes or cut-outs redrawn

Commit message: hw: V3.3 NFC 設定介面（ST25DV04KC＋板上印刷線圈），J5 改到左側板邊
- U6 ST25DV04KC（C3304276，ISO 15693＋I2C）；L5 板上線圈 14.9×14.6mm 8 圈 1.277µH，
  C22 75pF（C1681）→ 13.84MHz，C24 微調空位；I2C SDA=IO20、SCL=IO19，10k 上拉
- DI_1–4 改接 IO3/IO15/IO22/IO21（與 I2C 照左右順序排，佈線不交叉）
- J5 直立貼左側板邊，左半段上緣到 107.2mm，左上角給線圈
- upgrade_v32_pcb.py 以 WO_VER=3.2／3.3 切換；nfc_coil.py 以實際封裝銅箔算電感
- mains_router：禁布區外擴半線寬、禁止鋪銅的禁布區也擋、讀真實 L 形板框
- add_stitching --prune 也移除懸空 GND 過孔
- ERC 0；DRC 錯誤 0、未連線 0、parity 0；V3.2 用新程式重建仍為 0

Co-Authored-By: Claude Opus 5.5 (1M context) <noreply@anthropic.com>
Parts:
- added C22: 75pF C0G, Capacitor_SMD:C_0603_1608Metric, F.Cu at (115.9, 94.6)
- added C23: 100nF, Capacitor_SMD:C_0603_1608Metric, B.Cu at (124.0, 95.7)
- added C24: DNP trim, Capacitor_SMD:C_0603_1608Metric, F.Cu at (115.9, 96.9)
- added L5: NFC coil 1.27uH, WOOW:NFC_Coil_14.9x14.6mm_8T, F.Cu at (118.0, 83.7)
- added R24: 10k, Resistor_SMD:R_0603_1608Metric, B.Cu at (121.0, 95.1)
- added R25: 10k, Resistor_SMD:R_0603_1608Metric, B.Cu at (121.0, 97.5)
- added U6: ST25DV04KC-IE6S3, Package_SO:SOIC-8_3.9x4.9mm_P1.27mm, F.Cu at (121.4, 96.3)
- moved R18 14.4 mm to (104.8, 85.2)
- moved R23 13.3 mm to (102.0, 80.2), turned to 90 degrees
- moved R17 12.0 mm to (102.0, 88.7)
- moved J5 10.4 mm to (107.5, 88.7), turned to 90 degrees
- moved R16 4.88 mm to (104.8, 92.2)
- moved R15 4.56 mm to (102.0, 95.7)
Connections:
- U1 pad 17: /DI_4 -> /NFC_SCL
- U1 pad 18: /DI_3 -> /NFC_SDA
- U1 pad 19: /DI_2 -> /DI_4
- U1 pad 20: /DI_1 -> /DI_3
- U1 pad 23: unconnected-(U1-IO15-Pad23) -> /DI_2
- U1 pad 26: unconnected-(U1-IO3-Pad26) -> /DI_1
Routing:
- net /NFC_SDA: track 0.00 -> 44.1 mm, vias 0 -> 2
- net /NFC_SCL: track 0.00 -> 39.3 mm, vias 0 -> 2
- net /+3V3: track 125.2 -> 151.5 mm, vias 3 -> 7
- net /+12V_DI: track 2.60 -> 22.8 mm, vias 0 -> 1
- net /DI_A4: track 10.3 -> 25.5 mm
- net /DI_COM: track 19.5 -> 34.1 mm
- net /NFC_AC1: track 0.00 -> 12.6 mm, vias 0 -> 2
- net /NFC_AC0: track 0.00 -> 11.7 mm
- net /DI_A3: track 10.5 -> 20.9 mm, vias 0 -> 2
- net /DI_1: track 23.3 -> 29.6 mm, vias 1 -> 3
- net /DI_A2: track 10.9 -> 16.4 mm
- net /DI_2: track 26.2 -> 21.2 mm, vias 3 -> 1
- net /DI_A1: track 11.3 -> 15.2 mm
- net /DI_IN1: track 2.60 -> 6.08 mm
- net /DI_IN3: track 2.60 -> 6.08 mm
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Other:
- board size 63.4 x 93.1 mm -> 63.4 x 107.2 mm
